File: Hardware/Umweltdaten/LM75/LM75.sch (KiCad schematic (older format))
At the start: 6 parts, among them IC2 LM75, P1 I2C

Commit message: LM/TMP75 layout
Parts:
- added R1, R2, R3: 10k, Resistors_SMD:R_0805_HandSoldering, symbol R
Connections:
- net +3V3: now also R1.1, R2.1, R3.1
- net at IC2.1 (SDA), P1.2 (P2): now also R3.2
- net at IC2.2 (SCL), P1.3 (P3): now also R2.2
- net at IC2.3 (O.S.), P1.4 (P4): now also R1.2
Other:
- moved on the sheet: C1, IC2, JP1, JP2, JP3, P1
Changed lines of the file:
@@
 LIBS:contrib
 LIBS:valves
+LIBS:LM75-cache
 EELAYER 25 0
 EELAYER END
@@
 L LM75 IC2
 U 1 1 55D42F1C
-P 2600 2200
-F 0 "IC2" H 2350 2550 50  0000 C CNN
-F 1 "LM75" H 2800 1850 50  0000 C CNN
-F 2 "SMD_Packages:SOIC-8-N" H 2600 2150 50  0001 C CNN
-F 3 "" H 2600 2150 50  0000 C CNN
-	1    2600 2200
+P 4600 2700
+F 0 "IC2" H 4350 3050 50  0000 C CNN
+F 1 "LM75" H 4800 2350 50  0000 C CNN
+F 2 "SMD_Packages:SOIC-8-N" H 4600 2650 50  0001 C CNN
+F 3 "" H 4600 2650 50  0000 C CNN
+	1    4600 2700
 	1    0    0    -1
 $EndComp
@@
 L JUMPER3 JP1
 U 1 1 55D42F35
-P 3500 2100
-F 0 "JP1" H 3550 2000 50  0000 L CNN
-F 1 "A0" H 3500 2200 50  0000 C BNN
-F 2 "Footprints:SJ_2" H 3500 2100 60  0001 C CNN
-F 3 "" H 3500 2100 60  0000 C CNN
-	1    3500 2100
+P 5500 2600
+F 0 "JP1" H 5550 2500 50  0000 L CNN
+F 1 "A0" H 5500 2700 50  0000 C BNN
+F 2 "Footprints:SJ_2" H 5500 2600 60  0001 C CNN
+F 3 "" H 5500 2600 60  0000 C CNN
+	1    5500 2600
 	0    1    1    0
 $EndComp
@@
 L JUMPER3 JP2
 U 1 1 55D42F3C
-P 3900 2200
-F 0 "JP2" H 3950 2100 50  0000 L CNN
-F 1 "A1" H 3900 2300 50  0000 C BNN
-F 2 "Footprints:SJ_2" H 3900 2200 60  0001 C CNN
-F 3 "" H 3900 2200 60  0000 C CNN
-	1    3900 2200
+P 5900 2700
+F 0 "JP2" H 5950 2600 50  0000 L CNN
+F 1 "A1" H 5900 2800 50  0000 C BNN
+F 2 "Footprints:SJ_2" H 5900 2700 60  0001 C CNN
+F 3 "" H 5900 2700 60  0000 C CNN
+	1    5900 2700
 	0    1    1    0
 $EndComp
@@
 L JUMPER3 JP3
 U 1 1 55D42F43
-P 4200 2300
-F 0 "JP3" H 4250 2200 50  0000 L CNN
-F 1 "A2" H 4200 2400 50  0000 C BNN
-F 2 "Footprints:SJ_2" H 4200 2300 60  0001 C CNN
-F 3 "" H 4200 2300 60  0000 C CNN
-	1    4200 2300
+P 6200 2800
+F 0 "JP3" H 6250 2700 50  0000 L CNN
+F 1 "A2" H 6200 2900 50  0000 C BNN
+F 2 "Footprints:SJ_2" H 6200 2800 60  0001 C CNN
+F 3 "" H 6200 2800 60  0000 C CNN
+	1    6200 2800
 	0    1    1    0
 $EndComp
 Wire Wire Line
-	3400 2100 3100 2100
-Wire Wire Line
-	3800 2200 3100 2200
-Wire Wire Line
-	4100 2300 3100 2300
-Wire Wire Line
-	3500 1600 3500 1850
-Connection ~ 2600 1600
-Wire Wire Line
-	3900 1600 3900 1950
-Connection ~ 3500 1600
-Wire Wire Line
-	4200 1600 4200 2050
-Connection ~ 3900 1600
-Wire Wire Line
-	4200 2800 4200 2550
-Connection ~ 2600 2800
-Wire Wire Line
-	3500 2800 3500 2350
-Connection ~ 3500 2800
-Wire Wire Line
-	3900 2800 3900 2450
-Connection ~ 3900 2800
+	5400 2600 5100 2600
+Wire Wire Line
+	5800 2700 5100 2700
+Wire Wire Line
+	6100 2800 5100 2800
+Wire Wire Line
+	5500 2000 5500 2350
+Connection ~ 4600 2000
+Wire Wire Line
+	5900 2000 5900 2450
+Connection ~ 5500 2000
+Wire Wire Line
+	6200 2000 6200 2550
+Connection ~ 5900 2000
+Wire Wire Line
+	6200 3300 6200 3050
+Connection ~ 4600 3300
+Wire Wire Line
+	5500 3300 5500 2850
+Connection ~ 5500 3300
+Wire Wire Line
+	5900 3300 5900 2950
+Connection ~ 5900 3300
 $Comp
 L CONN_01X05 P1
 U 1 1 55FDCB45
-P 1500 2100
-F 0 "P1" H 1500 2400 50  0000 C CNN
-F 1 "I2C" V 1600 2100 50  0000 C CNN
-F 2 "Pin_Headers:Pin_Header_Straight_1x05" H 1500 2100 60  0001 C CNN
-F 3 "" H 1500 2100 60  0000 C CNN
-	1    1500 2100
+P 2900 2600
+F 0 "P1" H 2900 2900 50  0000 C CNN
+F 1 "I2C" V 3000 2600 50  0000 C CNN
+F 2 "Pin_Headers:Pin_Header_Straight_1x05" H 2900 2600 60  0001 C CNN
+F 3 "" H 2900 2600 60  0000 C CNN
+	1    2900 2600
 	-1   0    0    -1
 $EndComp
 Wire Wire Line
-	2100 2000 1700 2000
-Wire Wire Line
-	2100 2100 1700 2100
-Wire Wire Line
-	2100 2400 2000 2400
-Wire Wire Line
-	2000 2400 2000 2200
-Wire Wire Line
-	2000 2200 1700 2200
-Wire Wire Line
-	1700 1900 1900 1900
-Wire Wire Line
-	1900 1900 1900 1600
-Wire Wire Line
-	1100 1600 4200 1600
-Wire Wire Line
-	1900 2800 1900 2300
-Wire Wire Line
-	1900 2300 1700 2300
-Wire Wire Line
-	1100 2800 4200 2800
-Wire Wire Line
-	2600 1500 2600 1700
-Wire Wire Line
-	2600 2700 2600 2900
+	3100 2500 4100 2500
+Wire Wire Line
+	3100 2600 4100 2600
+Wire Wire Line
+	3100 2700 4000 2700
+Wire Wire Line
+	3300 2400 3100 2400
+Wire Wire Line
+	3300 2000 3300 2400
+Wire Wire Line
+	2500 2000 6200 2000
+Wire Wire Line
+	3300 3300 3300 2800
+Wire Wire Line
+	3300 2800 3100 2800
+Wire Wire Line
+	2500 3300 6200 3300
+Wire Wire Line
+	4600 1900 4600 2200
+Wire Wire Line
+	4600 3200 4600 3400
 $Comp
 L +3V3 #PWR01
 U 1 1 55FDD02B
-P 2600 1500
-F 0 "#PWR01" H 2600 1350 50  0001 C CNN
-F 1 "+3V3" H 2600 1640 50  0000 C CNN
-F 2 "" H 2600 1500 60  0000 C CNN
-F 3 "" H 2600 1500 60  0000 C CNN
-	1    2600 1500
+P 4600 1900
+F 0 "#PWR01" H 4600 1750 50  0001 C CNN
+F 1 "+3V3" H 4600 2040 50  0000 C CNN
+F 2 "" H 4600 1900 60  0000 C CNN
+F 3 "" H 4600 1900 60  0000 C CNN
+	1    4600 1900
 	1    0    0    -1
 $EndComp
@@
 L GND #PWR02
 U 1 1 55FDD08F
-P 2600 2900
-F 0 "#PWR02" H 2600 2650 50  0001 C CNN
-F 1 "GND" H 2600 2750 50  0000 C CNN
-F 2 "" H 2600 2900 60  0000 C CNN
-F 3 "" H 2600 2900 60  0000 C CNN
-	1    2600 2900
+P 4600 3400
+F 0 "#PWR02" H 4600 3150 50  0001 C CNN
+F 1 "GND" H 4600 3250 50  0000 C CNN
+F 2 "" H 4600 3400 60  0000 C CNN
+F 3 "" H 4600 3400 60  0000 C CNN
+	1    4600 3400
 	1    0    0    -1
 $EndComp
@@
 L C C1
 U 1 1 55FDD272
-P 1100 2150
-F 0 "C1" H 1125 2250 50  0000 L CNN
-F 1 "100nF" H 1125 2050 50  0000 L CNN
-F 2 "Capacitors_SMD:C_0805_HandSoldering" H 1138 2000 30  0001 C CNN
-F 3 "" H 1100 2150 60  0000 C CNN
-	1    1100 2150
-	1    0    0    -1
-$EndComp
-Wire Wire Line
-	1100 2000 1100 1600
-Connection ~ 1900 1600
-Wire Wire Line
-	1100 2300 1100 2800
-Connection ~ 1900 2800
+P 2500 2650
+F 0 "C1" H 2525 2750 50  0000 L CNN
+F 1 "100nF" H 2525 2550 50  0000 L CNN
+F 2 "Capacitors_SMD:C_0805_HandSoldering" H 2538 2500 30  0001 C CNN
+F 3 "" H 2500 2650 60  0000 C CNN
+	1    2500 2650
+	1    0    0    -1
+$EndComp
+Wire Wire Line
+	2500 2000 2500 2500
+Connection ~ 3300 2000
+Wire Wire Line
+	2500 2800 2500 3300
+Connection ~ 3300 3300
+$Comp
+L R R3
+U 1 1 571CD6B6
+P 4000 2250
+F 0 "R3" V 4080 2250 50  0000 C CNN
+F 1 "10k" V 4000 2250 50  0000 C CNN
+F 2 "Resistors_SMD:R_0805_HandSoldering" V 3930 2250 50  0001 C CNN
+F 3 "" H 4000 2250 50  0000 C CNN
+	1    4000 2250
+	1    0    0    -1
+$EndComp
+$Comp
+L R R2
+U 1 1 571CD7A0
+P 3800 2250
+F 0 "R2" V 3880 2250 50  0000 C CNN
+F 1 "10k" V 3800 2250 50  0000 C CNN
+F 2 "Resistors_SMD:R_0805_HandSoldering" V 3730 2250 50  0001 C CNN
+F 3 "" H 3800 2250 50  0000 C CNN
+	1    3800 2250
+	1    0    0    -1
+$EndComp
+$Comp
+L R R1
+U 1 1 571CD7D0
+P 3600 2250
+F 0 "R1" V 3680 2250 50  0000 C CNN
+F 1 "10k" V 3600 2250 50  0000 C CNN
+F 2 "Resistors_SMD:R_0805_HandSoldering" V 3530 2250 50  0001 C CNN
+F 3 "" H 3600 2250 50  0000 C CNN
+	1    3600 2250
+	1    0    0    -1
+$EndComp
+Wire Wire Line
+	4000 2400 4000 2500
+Connection ~ 4000 2500
+Wire Wire Line
+	3800 2400 3800 2600
+Connection ~ 3800 2600
+Wire Wire Line
+	4000 2700 4000 2900
+Wire Wire Line
+	4000 2900 4100 2900
+Wire Wire Line
+	3600 2400 3600 2700
+Connection ~ 3600 2700
+Wire Wire Line
+	4000 2100 4000 2000
+Connection ~ 4000 2000
+Wire Wire Line
+	3800 2100 3800 2000
+Connection ~ 3800 2000
+Wire Wire Line
+	3600 2100 3600 2000
+Connection ~ 3600 2000
 $EndSCHEMATC

Commit message: finished LM/TMP75 PCB
Parts:
- P1: footprint Pin_Headers:Pin_Header_Straight_1x05 -> SMD:SMD_05-4mm
Changed lines of the file:
@@
 F 0 "P1" H 2900 2900 50  0000 C CNN
 F 1 "I2C" V 3000 2600 50  0000 C CNN
-F 2 "Pin_Headers:Pin_Header_Straight_1x05" H 2900 2600 60  0001 C CNN
+F 2 "SMD:SMD_05-4mm" H 2900 2600 60  0001 C CNN
 F 3 "" H 2900 2600 60  0000 C CNN
 	1    2900 2600
